Commit message: experiments for mdpi paper

File: src/pkg/rover_description_pkg/urdf/rover_gazebo.xacro (robot description, xacro)
@@ -117,5 +117,5 @@
     </xacro:sensor_d435i>  -->
     <joint name="camera_to_payload" type="fixed">
-        <origin xyz="0.1 0.0 0.04" rpy="0 0 0"/>
+        <origin xyz="0.1 0.0 0.1" rpy="0 0 0"/>
         <parent link="payload_link"/>
         <child link="${camera_base_frame}"/>

File: src/pkg/rover_description_pkg/urdf/rover_macro.xacro (robot description, xacro)
@@ -95,5 +95,5 @@
             <parent link="payload_link"/>
             <child link="${laser_frame}"/>
-            <origin xyz="0.075 0 0.035" rpy="0 3.1415 0.0"/>
+            <origin xyz="0.0 0.0 0.16" rpy="0.0 0.0 0.0"/>
         </joint>
         <link name="${laser_frame}">
