Commit message: experiment setup

File: src/pkg/rover_description_pkg/urdf/rover_macro.xacro (robot description, xacro)
@@ -95,5 +95,5 @@
             <parent link="payload_link"/>
             <child link="${laser_frame}"/>
-            <origin xyz="0.0 0.0 0.16" rpy="0.0 0.0 0.0"/>
+            <origin xyz="0.0 0.0 0.14" rpy="0.0 0.0 0.0"/>
         </joint>
         <link name="${laser_frame}">
@@ -105,5 +105,5 @@
             </visual>
             <collision>
-                <origin xyz="0 0 -0.05" rpy="0 0 3.1415"/>
+                <origin xyz="0 0 0.0" rpy="0 0 3.1415"/>
                 <geometry>
                     <cylinder radius="0.05" length="0.15"/>
